Commit message: [ADD] DG-4F & Safely Send Duty

File: dg4f_driver/urdf/dg4f_ros2_control.xacro (robot description, xacro)
@@ -1,37 +1,36 @@
 <?xml version="1.0"?>
 <robot name="delto_5f" xmlns:xacro="http://www.ros.org/wiki/xacro">
-    <xacro:include filename="$(find dg_description)/urdf/dg5f_left.xacro" />
+    <xacro:include filename="$(find dg_description)/urdf/dg4f.urdf" />
     <link name="base_link" />
     <joint name="base_joint" type="fixed">
         <parent link="base_link" />
-        <child link="left_base_link" />
+        <child link="l_dg_mount" />
         <origin xyz="0 0 0" rpy="0 0 0" />
     </joint>
-    <ros2_control name="dg5f_driver" type="system">
+    <ros2_control name="dg4f_driver" type="system">
         <hardware>
-            <plugin>dg5f_driver/SystemInterface</plugin>
+            <plugin>dg4f_driver/SystemInterface</plugin>
+            <!-- GripperOption -->
             <param name="delto_ip">$(arg delto_ip)</param>
             <param name="delto_port">$(arg delto_port)</param>
-            <param name="delto_model">24338</param>
-            <param name="hand_type">left</param>
-            <!-- <param name="firmware_version">$(arg firmware_version)</param> -->
+            <param name="delto_model">20226</param> <!-- 0x4F02 -->
         </hardware>
         <!-- Finger 1 joints -->
-        <joint name="lj_dg_1_1">
+        <joint name="j_dg_1_1">
             <command_interface name="effort" />
             <state_interface name="position" />
             <state_interface name="velocity" />
         </joint>
-        <joint name="lj_dg_1_2">
+        <joint name="j_dg_1_2">
             <command_interface name="effort" />
             <state_interface name="position" />
             <state_interface name="velocity" />
         </joint>
-        <joint name="lj_dg_1_3">
+        <joint name="j_dg_1_3">
             <command_interface name="effort" />
             <state_interface name="position" />
             <state_interface name="velocity" />
         </joint>
-        <joint name="lj_dg_1_4">
+        <joint name="j_dg_1_4">
             <command_interface name="effort" />
             <state_interface name="position" />
@@ -39,20 +38,20 @@
         </joint>
         <!-- Finger 2 joints -->
-        <joint name="lj_dg_2_1">
+        <joint name="j_dg_2_1">
             <command_interface name="effort" />
             <state_interface name="position" />
             <state_interface name="velocity" />
         </joint>
-        <joint name="lj_dg_2_2">
+        <joint name="j_dg_2_2">
             <command_interface name="effort" />
             <state_interface name="position" />
             <state_interface name="velocity" />
         </joint>
-        <joint name="lj_dg_2_3">
+        <joint name="j_dg_2_3">
             <command_interface name="effort" />
             <state_interface name="position" />
             <state_interface name="velocity" />
         </joint>
-        <joint name="lj_dg_2_4">
+        <joint name="j_dg_2_4">
             <command_interface name="effort" />
             <state_interface name="position" />
@@ -60,20 +59,20 @@
         </joint>
         <!-- Finger 3 joints -->
-        <joint name="lj_dg_3_1">
+        <joint name="j_dg_3_1">
             <command_interface name="effort" />
             <state_interface name="position" />
             <state_interface name="velocity" />
         </joint>
-        <joint name="lj_dg_3_2">
+        <joint name="j_dg_3_2">
             <command_interface name="effort" />
             <state_interface name="position" />
             <state_interface name="velocity" />
         </joint>
-        <joint name="lj_dg_3_3">
+        <joint name="j_dg_3_3">
             <command_interface name="effort" />
             <state_interface name="position" />
             <state_interface name="velocity" />
         </joint>
-        <joint name="lj_dg_3_4">
+        <joint name="j_dg_3_4">
             <command_interface name="effort" />
             <state_interface name="position" />
@@ -81,41 +80,30 @@
         </joint>
         <!-- Finger 4 joints -->
-        <joint name="lj_dg_4_1">
+         <joint name="j_dg_4_1">
             <command_interface name="effort" />
             <state_interface name="position" />
             <state_interface name="velocity" />
         </joint>
-        <joint name="lj_dg_4_2">
+        <joint name="j_dg_4_2">
             <command_interface name="effort" />
             <state_interface name="position" />
             <state_interface name="velocity" />
         </joint>
-        <joint name="lj_dg_4_3">
+        <joint name = "j_dg_4_3">
             <command_interface name="effort" />
             <state_interface name="position" />
             <state_interface name="velocity" />
         </joint>
-        <joint name="lj_dg_4_4">
+        <joint name = "j_dg_4_4">
             <command_interface name="effort" />
             <state_interface name="position" />
             <state_interface name="velocity" />
         </joint>
-        <!-- Finger 5 joints -->
-        <joint name="lj_dg_5_1">
+        <joint name = "j_dg_1_inner">
             <command_interface name="effort" />
             <state_interface name="position" />
             <state_interface name="velocity" />
         </joint>
-        <joint name="lj_dg_5_2">
-            <command_interface name="effort" />
-            <state_interface name="position" />
-            <state_interface name="velocity" />
-        </joint>
-        <joint name="lj_dg_5_3">
-            <command_interface name="effort" />
-            <state_interface name="position" />
-            <state_interface name="velocity" />
-        </joint>
-        <joint name="lj_dg_5_4">
+        <joint name = "j_dg_4_inner">
             <command_interface name="effort" />
             <state_interface name="position" />

File: dg5f_driver/urdf/dg5f_right_ros2_control.xacro (robot description, xacro)
@@ -13,4 +13,5 @@
             <param name="delto_ip">$(arg delto_ip)</param>
             <param name="delto_port">$(arg delto_port)</param>
+             <!-- <param name="firmware_version">$(arg firmware_version)</param> -->
             <param name="delto_model">24354</param>
             <param name="hand_type">right</param>

Commit message: refactor: refactor dg4f_driver package
- Migrate hardware interface to shared delto_hardware package
- Add effort controller configuration
- Add fingertip F/T sensor broadcaster support
- Add new launch files (dg4f_driver, dg4f_effort_controller)
- Add PID controller test scripts
- Remove duplicated hardware interface code
- Update package dependencies

File: dg4f_driver/urdf/dg4f_ros2_control.xacro (robot description, xacro)
@@ -1,4 +1,9 @@
 <?xml version="1.0"?>
 <robot name="delto_5f" xmlns:xacro="http://www.ros.org/wiki/xacro">
+    <!-- Default argument values -->
+    <xacro:arg name="delto_ip" default="169.254.186.72" />
+    <xacro:arg name="delto_port" default="502" />
+    <xacro:arg name="fingertip_sensor" default="false" />
+    <xacro:arg name="io" default="false" />
     <xacro:include filename="$(find dg_description)/urdf/dg4f.urdf" />
     <link name="base_link" />
@@ -8,11 +13,41 @@
         <origin xyz="0 0 0" rpy="0 0 0" />
     </joint>
+    <!-- Fingertip F/T sensor frames -->
+    <!-- Finger 1 -->
+    <link name="fingertip_1" />
+    <joint name="fingertip_1_joint" type="fixed">
+        <parent link="l_dg_1_tip" />
+        <child link="fingertip_1" />
+        <origin xyz="0 0 0" rpy="0 0 0" />
+    </joint>
+    <!-- Finger 2 -->
+    <link name="fingertip_2" />
+    <joint name="fingertip_2_joint" type="fixed">
+        <parent link="l_dg_2_tip" />
+        <child link="fingertip_2" />
+        <origin xyz="0 0 0" rpy="0 0 0" />
+    </joint>
+    <!-- Finger 3 -->
+    <link name="fingertip_3" />
+    <joint name="fingertip_3_joint" type="fixed">
+        <parent link="l_dg_3_tip" />
+        <child link="fingertip_3" />
+        <origin xyz="0 0 0" rpy="0 0 0" />
+    </joint>
+    <!-- Finger 4 -->
+    <link name="fingertip_4" />
+    <joint name="fingertip_4_joint" type="fixed">
+        <parent link="l_dg_4_tip" />
+        <child link="fingertip_4" />
+        <origin xyz="0 0 0" rpy="0 0 0" />
+    </joint>
     <ros2_control name="dg4f_driver" type="system">
         <hardware>
-            <plugin>dg4f_driver/SystemInterface</plugin>
-            <!-- GripperOption -->
+            <plugin>delto_hardware/SystemInterface</plugin>
             <param name="delto_ip">$(arg delto_ip)</param>
             <param name="delto_port">$(arg delto_port)</param>
             <param name="delto_model">20226</param> <!-- 0x4F02 -->
+            <param name="fingertip_sensor">$(arg fingertip_sensor)</param>
+            <param name="IO">$(arg io)</param>
         </hardware>
         <!-- Finger 1 joints -->
@@ -110,4 +145,17 @@
             <state_interface name="velocity" />
         </joint>
+        <!-- FT sensors for each finger (4f) -->
+        <sensor name="fingertip_finger_1" type="force_torque">
+            <param name="frame_id">fingertip_1</param>
+        </sensor>
+        <sensor name="fingertip_finger_2" type="force_torque">
+            <param name="frame_id">fingertip_2</param>
+        </sensor>
+        <sensor name="fingertip_finger_3" type="force_torque">
+            <param name="frame_id">fingertip_3</param>
+        </sensor>
+        <sensor name="fingertip_finger_4" type="force_torque">
+            <param name="frame_id">fingertip_4</param>
+        </sensor>
     </ros2_control>
 </robot>
