Commit message: refactor: refactor dg5f_driver package
- Migrate hardware interface to shared delto_hardware package
- Add effort controller configurations for left/right hands
- Add fingertip F/T sensor broadcaster support (left/right/both)
- Add new PID controller launch files
- Add both hands PID all controller launch
- Add joint trajectory controller test scripts
- Add manus glove retargeting script
- Remove duplicated hardware interface code
- Update package dependencies

File: dg5f_driver/urdf/dg5f_both_ros2_control.xacro (robot description, xacro)
@@ -1,30 +1,93 @@
 <?xml version="1.0"?>
 <robot name="delto_5f" xmlns:xacro="http://www.ros.org/wiki/xacro">
+    <!-- Default argument values -->
+    <xacro:arg name="dg5f_right_ip" default="192.168.31.72" />
+    <xacro:arg name="dg5f_right_port" default="502" />
+    <xacro:arg name="dg5f_right_model" default="24354" />
+    <xacro:arg name="dg5f_left_ip" default="192.168.31.73" />
+    <xacro:arg name="dg5f_left_port" default="502" />
+    <xacro:arg name="dg5f_left_model" default="24354" />
+    <xacro:arg name="fingertip_sensor" default="false" />
+    <xacro:arg name="io" default="false" />
+    <xacro:include filename="$(find dg_description)/urdf/dg5f_left.xacro" />
     <xacro:include filename="$(find dg_description)/urdf/dg5f_right.xacro" />
-    <xacro:include filename="$(find dg_description)/urdf/dg5f_left.xacro" />
     <link name="base_link" />
     <joint name="base_joint" type="fixed">
         <parent link="base_link" />
-        <child link="right_base_link" />
-        <origin xyz="0.15 0 0" rpy="0 0 0" />
-    </joint>
-    <joint name="left_base_joint" type="fixed">
-        <parent link="base_link" />
         <child link="left_base_link" />
-        <origin xyz="-0.15 0 0" rpy="0 0 0" />
-    </joint>
-  <xacro:arg name="dg5f_right_ip" default="192.168.31.72" />
-  <xacro:arg name="dg5f_right_port" default="502" />
-  <xacro:arg name="dg5f_right_model" default="24354" />
-  <xacro:arg name="dg5f_left_ip" default="192.168.31.73" />
-  <xacro:arg name="dg5f_left_port" default="502" />
-  <xacro:arg name="dg5f_left_model" default="24354" />
+        <origin xyz="0 0 0" rpy="0 0 0" />
+    </joint>
+    <!-- Left Hand Fingertip F/T sensor frames -->
+    <link name="left_fingertip_1" />
+    <joint name="left_fingertip_1_joint" type="fixed">
+        <parent link="ll_dg_1_tip" />
+        <child link="left_fingertip_1" />
+        <origin xyz="0 -0.015 0" rpy="0 0 0" />
+    </joint>
+    <link name="left_fingertip_2" />
+    <joint name="left_fingertip_2_joint" type="fixed">
+        <parent link="ll_dg_2_tip" />
+        <child link="left_fingertip_2" />
+        <origin xyz="0 -0.015 0" rpy="0 0 0" />
+    </joint>
+    <link name="left_fingertip_3" />
+    <joint name="left_fingertip_3_joint" type="fixed">
+        <parent link="ll_dg_3_tip" />
+        <child link="left_fingertip_3" />
+        <origin xyz="0 -0.015 0" rpy="0 0 0" />
+    </joint>
+    <link name="left_fingertip_4" />
+    <joint name="left_fingertip_4_joint" type="fixed">
+        <parent link="ll_dg_4_tip" />
+        <child link="left_fingertip_4" />
+        <origin xyz="0 -0.015 0" rpy="0 0 0" />
+    </joint>
+    <link name="left_fingertip_5" />
+    <joint name="left_fingertip_5_joint" type="fixed">
+        <parent link="ll_dg_5_tip" />
+        <child link="left_fingertip_5" />
+        <origin xyz="0 -0.015 0" rpy="0 0 0" />
+    </joint>
+    <!-- Right Hand Fingertip F/T sensor frames -->
+    <link name="right_fingertip_1" />
+    <joint name="right_fingertip_1_joint" type="fixed">
+        <parent link="rl_dg_1_tip" />
+        <child link="right_fingertip_1" />
+        <origin xyz="0 -0.015 0" rpy="0 0 0" />
+    </joint>
+    <link name="right_fingertip_2" />
+    <joint name="right_fingertip_2_joint" type="fixed">
+        <parent link="rl_dg_2_tip" />
+        <child link="right_fingertip_2" />
+        <origin xyz="0 -0.015 0" rpy="0 0 0" />
+    </joint>
+    <link name="right_fingertip_3" />
+    <joint name="right_fingertip_3_joint" type="fixed">
+        <parent link="rl_dg_3_tip" />
+        <child link="right_fingertip_3" />
+        <origin xyz="0 -0.015 0" rpy="0 0 0" />
+    </joint>
+    <link name="right_fingertip_4" />
+    <joint name="right_fingertip_4_joint" type="fixed">
+        <parent link="rl_dg_4_tip" />
+        <child link="right_fingertip_4" />
+        <origin xyz="0 -0.015 0" rpy="0 0 0" />
+    </joint>
+    <link name="right_fingertip_5" />
+    <joint name="right_fingertip_5_joint" type="fixed">
+        <parent link="rl_dg_5_tip" />
+        <child link="right_fingertip_5" />
+        <origin xyz="0 -0.015 0" rpy="0 0 0" />
+    </joint>
+  <!-- DG5F Right gripper hardware -->
   <ros2_control name="DG5FRightHardware" type="system">
     <hardware>
-      <plugin>dg5f_driver/SystemInterface</plugin>
+      <plugin>delto_hardware/SystemInterface</plugin>
       <param name="delto_ip">$(arg dg5f_right_ip)</param>
       <param name="delto_port">$(arg dg5f_right_port)</param>
       <param name="delto_model">$(arg dg5f_right_model)</param>
       <param name="hand_type">right</param>
+      <param name="fingertip_sensor">$(arg fingertip_sensor)</param>
+      <param name="IO">$(arg io)</param>
     </hardware>
     <!-- Finger 1 joints -->
@@ -137,9 +200,11 @@
   <ros2_control name="DG5FLeftHardware" type="system">
     <hardware>
-      <plugin>dg5f_driver/SystemInterface</plugin>
+      <plugin>delto_hardware/SystemInterface</plugin>
       <param name="delto_ip">$(arg dg5f_left_ip)</param>
       <param name="delto_port">$(arg dg5f_left_port)</param>
       <param name="delto_model">$(arg dg5f_left_model)</param>
       <param name="hand_type">left</param>
+      <param name="fingertip_sensor">$(arg fingertip_sensor)</param>
+      <param name="IO">$(arg io)</param>
     </hardware>
     <!-- Finger 1 joints -->

File: dg5f_driver/urdf/dg5f_left_ros2_control.xacro (robot description, xacro)
@@ -1,4 +1,9 @@
 <?xml version="1.0"?>
 <robot name="delto_5f" xmlns:xacro="http://www.ros.org/wiki/xacro">
+    <!-- Default argument values -->
+    <xacro:arg name="delto_ip" default="169.254.186.73" />
+    <xacro:arg name="delto_port" default="502" />
+    <xacro:arg name="fingertip_sensor" default="false" />
+    <xacro:arg name="io" default="false" />
     <xacro:include filename="$(find dg_description)/urdf/dg5f_left.xacro" />
     <link name="base_link" />
@@ -8,12 +13,49 @@
         <origin xyz="0 0 0" rpy="0 0 0" />
     </joint>
+    <!-- Fingertip F/T sensor frames -->
+    <!-- Finger 1 (Thumb) -->
+    <link name="left_fingertip_1" />
+    <joint name="left_fingertip_1_joint" type="fixed">
+        <parent link="ll_dg_1_tip" />
+        <child link="left_fingertip_1" />
+        <origin xyz="0 0 0" rpy="0 1.5708 0" />
+    </joint>
+    <!-- Finger 2 (Index) -->
+    <link name="left_fingertip_2" />
+    <joint name="left_fingertip_2_joint" type="fixed">
+        <parent link="ll_dg_2_tip" />
+        <child link="left_fingertip_2" />
+        <origin xyz="0 0 0" rpy="0 1.5708 0" />
+    </joint>
+    <!-- Finger 3 (Middle) -->
+    <link name="left_fingertip_3" />
+    <joint name="left_fingertip_3_joint" type="fixed">
+        <parent link="ll_dg_3_tip" />
+        <child link="left_fingertip_3" />
+        <origin xyz="0 0 0" rpy="0 1.5708 0" />
+    </joint>
+    <!-- Finger 4 (Ring) -->
+    <link name="left_fingertip_4" />
+<joint name="left_fingertip_4_joint" type="fixed">
+        <parent link="ll_dg_4_tip" />
+    <child link="left_fingertip_4" />
+        <origin xyz="0 0 0" rpy="0 1.5708 0" />
+    </joint>
+<!-- Finger 5 (Pinky) -->
+    <link name="left_fingertip_5" />
+    <joint name="left_fingertip_5_joint" type="fixed">
+        <parent link="ll_dg_5_tip" />
+    <child link="left_fingertip_5" />
+        <origin xyz="0 0 0" rpy="0 1.5708 0" />
+    </joint>
     <ros2_control name="dg5f_driver" type="system">
         <hardware>
-            <plugin>dg5f_driver/SystemInterface</plugin>
+            <plugin>delto_hardware/SystemInterface</plugin>
             <param name="delto_ip">$(arg delto_ip)</param>
             <param name="delto_port">$(arg delto_port)</param>
             <param name="delto_model">24338</param>
             <param name="hand_type">left</param>
-            <!-- <param name="firmware_version">$(arg firmware_version)</param> -->
+            <param name="fingertip_sensor">$(arg fingertip_sensor)</param>
+            <param name="IO">$(arg io)</param>
         </hardware>
         <!-- Finger 1 joints -->

File: dg5f_driver/urdf/dg5f_right_ros2_control.xacro (robot description, xacro)
@@ -1,4 +1,9 @@
 <?xml version="1.0"?>
 <robot name="delto_5f" xmlns:xacro="http://www.ros.org/wiki/xacro">
+    <!-- Default argument values -->
+    <xacro:arg name="delto_ip" default="169.254.186.72" />
+    <xacro:arg name="delto_port" default="502" />
+    <xacro:arg name="fingertip_sensor" default="false" />
+    <xacro:arg name="io" default="false" />
     <xacro:include filename="$(find dg_description)/urdf/dg5f_right.xacro" />
     <link name="base_link" />
@@ -8,12 +13,49 @@
         <origin xyz="0 0 0" rpy="0 0 0" />
     </joint>
+    <!-- Fingertip F/T sensor frames -->
+    <!-- Finger 1 (Thumb) -->
+    <link name="right_fingertip_1" />
+    <joint name="right_fingertip_1_joint" type="fixed">
+        <parent link="rl_dg_1_tip" />
+        <child link="right_fingertip_1" />
+        <origin xyz="0 0 0" rpy="0 0 -1.5708" />
+    </joint>
+    <!-- Finger 2 (Index) -->
+    <link name="right_fingertip_2" />
+    <joint name="right_fingertip_2_joint" type="fixed">
+        <parent link="rl_dg_2_tip" />
+        <child link="right_fingertip_2" />
+        <origin xyz="0 0 0" rpy="0 1.5708 0" />
+    </joint>
+    <!-- Finger 3 (Middle) -->
+    <link name="right_fingertip_3" />
+    <joint name="right_fingertip_3_joint" type="fixed">
+        <parent link="rl_dg_3_tip" />
+        <child link="right_fingertip_3" />
+        <origin xyz="0 0 0" rpy="0 1.5708 0" />
+    </joint>
+    <!-- Finger 4 (Ring) -->
+    <link name="right_fingertip_4" />
+    <joint name="right_fingertip_4_joint" type="fixed">
+        <parent link="rl_dg_4_tip" />
+        <child link="right_fingertip_4" />
+        <origin xyz="0 0 0" rpy="0 1.5708 0" />
+    </joint>
+    <!-- Finger 5 (Pinky) -->
+    <link name="right_fingertip_5" />
+    <joint name="right_fingertip_5_joint" type="fixed">
+        <parent link="rl_dg_5_tip" />
+        <child link="right_fingertip_5" />
+        <origin xyz="0 0 0" rpy="0 1.5708 0" />
+    </joint>
     <ros2_control name="dg5f_driver" type="system">
         <hardware>
-            <plugin>dg5f_driver/SystemInterface</plugin>
+            <plugin>delto_hardware/SystemInterface</plugin>
             <param name="delto_ip">$(arg delto_ip)</param>
             <param name="delto_port">$(arg delto_port)</param>
-             <!-- <param name="firmware_version">$(arg firmware_version)</param> -->
             <param name="delto_model">24354</param>
             <param name="hand_type">right</param>
+            <param name="fingertip_sensor">$(arg fingertip_sensor)</param>
+            <param name="IO">$(arg io)</param>
         </hardware>
         <!-- Finger 1 joints -->
