Commit message: feat:update sensor tip in urdf and xacro.

File: dg5f_driver/urdf/dg5f_right_ros2_control.xacro (robot description, xacro)
@@ -1,58 +1,77 @@
 <?xml version="1.0"?>
-<robot name="delto_5f" xmlns:xacro="http://www.ros.org/wiki/xacro">
+<robot name="dg5f_right" xmlns:xacro="http://www.ros.org/wiki/xacro">
     <!-- Default argument values -->
     <xacro:arg name="delto_ip" default="169.254.186.72" />
     <xacro:arg name="delto_port" default="502" />
+    <xacro:arg name="delto_model" default="24354" />
     <xacro:arg name="fingertip_sensor" default="false" />
     <xacro:arg name="io" default="false" />
-    <xacro:include filename="$(find dg_description)/urdf/dg5f_right.xacro" />
+    <!-- DG5F arguments -->
+    <xacro:arg name="base_type" default="default" />
+    <xacro:arg name="with_mount" default="true" />
+    <!-- Tip type is determined by fingertip_sensor -->
+    <xacro:property name="fs" value="$(arg fingertip_sensor)" />
+    <xacro:property name="tip_type" value="${'type1' if str(fs).lower() == 'true' else 'default'}" />
+    <!-- Include dg5f_macro.xacro (macro only, no standalone instantiation) -->
+    <xacro:include filename="$(find dg_description)/urdf/dg5f_macro.xacro" />
+    <!-- Base link -->
     <link name="base_link" />
     <joint name="base_joint" type="fixed">
         <parent link="base_link" />
-        <child link="right_base_link" />
+        <child link="rl_dg_base_link" />
         <origin xyz="0 0 0" rpy="0 0 0" />
     </joint>
-    <!-- Fingertip F/T sensor frames -->
-    <!-- Finger 1 (Thumb) -->
-    <link name="right_fingertip_1" />
-    <joint name="right_fingertip_1_joint" type="fixed">
-        <parent link="rl_dg_1_tip" />
-        <child link="right_fingertip_1" />
-        <origin xyz="0 0 0" rpy="0 0 -1.5708" />
-    </joint>
-    <!-- Finger 2 (Index) -->
-    <link name="right_fingertip_2" />
-    <joint name="right_fingertip_2_joint" type="fixed">
-        <parent link="rl_dg_2_tip" />
-        <child link="right_fingertip_2" />
-        <origin xyz="0 0 0" rpy="0 1.5708 0" />
-    </joint>
-    <!-- Finger 3 (Middle) -->
-    <link name="right_fingertip_3" />
-    <joint name="right_fingertip_3_joint" type="fixed">
-        <parent link="rl_dg_3_tip" />
-        <child link="right_fingertip_3" />
-        <origin xyz="0 0 0" rpy="0 1.5708 0" />
-    </joint>
-    <!-- Finger 4 (Ring) -->
-    <link name="right_fingertip_4" />
-    <joint name="right_fingertip_4_joint" type="fixed">
-        <parent link="rl_dg_4_tip" />
-        <child link="right_fingertip_4" />
-        <origin xyz="0 0 0" rpy="0 1.5708 0" />
-    </joint>
-    <!-- Finger 5 (Pinky) -->
-    <link name="right_fingertip_5" />
-    <joint name="right_fingertip_5_joint" type="fixed">
-        <parent link="rl_dg_5_tip" />
-        <child link="right_fingertip_5" />
-        <origin xyz="0 0 0" rpy="0 1.5708 0" />
-    </joint>
-    <ros2_control name="dg5f_driver" type="system">
+    <!-- Instantiate right hand -->
+    <xacro:dg5f_hand
+        side="right"
+        base_type="$(arg base_type)"
+        with_mount="$(arg with_mount)"
+        tip1_type="${tip_type}"
+        tip2_type="${tip_type}"
+        tip3_type="${tip_type}"
+        tip4_type="${tip_type}"
+        tip5_type="${tip_type}"
+    />
+    <!-- Fingertip F/T sensor frames (only when fingertip_sensor is true) -->
+    <xacro:if value="${str(fs).lower() == 'true'}">
+        <link name="right_fingertip_1" />
+        <joint name="right_fingertip_1_joint" type="fixed">
+            <parent link="rl_dg_1_tip" />
+            <child link="right_fingertip_1" />
+            <origin xyz="0 0.0128 0.0045" rpy="0 0 -1.5708" />
+        </joint>
+        <link name="right_fingertip_2" />
+        <joint name="right_fingertip_2_joint" type="fixed">
+            <parent link="rl_dg_2_tip" />
+            <child link="right_fingertip_2" />
+            <origin xyz="0.0045 0 0.0128" rpy="0 1.5708 0" />
+        </joint>
+        <link name="right_fingertip_3" />
+        <joint name="right_fingertip_3_joint" type="fixed">
+            <parent link="rl_dg_3_tip" />
+            <child link="right_fingertip_3" />
+            <origin xyz="0.0045 0 0.0128" rpy="0 1.5708 0" />
+        </joint>
+        <link name="right_fingertip_4" />
+        <joint name="right_fingertip_4_joint" type="fixed">
+            <parent link="rl_dg_4_tip" />
+            <child link="right_fingertip_4" />
+            <origin xyz="0.0045 0 0.0128" rpy="0 1.5708 0" />
+        </joint>
+        <link name="right_fingertip_5" />
+        <joint name="right_fingertip_5_joint" type="fixed">
+            <parent link="rl_dg_5_tip" />
+            <child link="right_fingertip_5" />
+            <origin xyz="0.0045 0 0.0128" rpy="0 1.5708 0" />
+        </joint>
+    </xacro:if>
+    <!-- ROS2 Control -->
+    <ros2_control name="DG5FRightHardware" type="system">
         <hardware>
-            <plugin>delto_hardware/SystemInterface</plugin>
+            <plugin>mock_components/GenericSystem</plugin>
+            <!-- <plugin>delto_hardware/SystemInterface</plugin> -->
             <param name="delto_ip">$(arg delto_ip)</param>
             <param name="delto_port">$(arg delto_port)</param>
-            <param name="delto_model">24354</param>
+            <param name="delto_model">$(arg delto_model)</param>
             <param name="hand_type">right</param>
             <param name="fingertip_sensor">$(arg fingertip_sensor)</param>
