Commit message: Add inertial properties to l_dg_mount link in URDF and XACRO files

File: dg_description/urdf/dg3f_m.xacro (robot description, xacro)
@@ -17,4 +17,6 @@
   <link name="l_dg_mount">
     <inertial>
+      <origin xyz="6.4721E-09 2.1674E-05 0.0049997" rpy="0.0 0.0 0.0" />
+      <inertia ixx="1.0999E-05" ixy="-2.1734E-12" ixz="-1.2441E-12" iyy="1.1018E-05" iyz="-4.0435E-09" izz="2.0531E-05" />
       <mass value="0.035" />
     </inertial>
